File: ArmonicWaveLevitationV2/ArmonicWaveLevitation.kicad_pcb (KiCad board)
At the start: 2 copper layers, 27 x 27 mm, 17 parts, among them J1 Batt conn, J6 SPK, SW1 POW, U1 TC78H621FNG, U2 LM78L05_TO92, U3 NA555D

Commit message: u
Routing:
- net 40KHz: track 0.00 -> 15.7 mm, vias 0 -> 3
- net +5V: track 36.9 -> 37.6 mm
